File: hardware/calc/calc.kicad_sch (KiCad schematic)
At the start: 30 parts, among them J1 BAT, Q1 AP3101, SW17 MSK12C02, U3 TP4056 Module 28x17

Commit message: updated kicad files
Parts:
- Q1: value AP3101 -> AP3401
Changed lines of the file:
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@@
       (effects (font (size 1.27 1.27)))
     )
-    (property "Value" "AP3101" (at 226.06 38.1 90)
+    (property "Value" "AP3401" (at 226.06 38.1 90)
       (effects (font (size 1.27 1.27)))
     )
